Commit message: initial commit

File: surrol/assets/gauze/gauze.urdf (robot description, URDF)
Before this commit: robot sphere, 1 links, 0 joints
Links:
- link baseLink: geometry collision box size=0.004 0.002 0.003; visual mesh filename=meshes/gauze.obj scale=2 2 2

File: surrol/assets/needle/needle_shapes.urdf (robot description, URDF)
Before this commit: robot needle, 7 links, 6 joints
Links:
- link baseLink: geometry collision mesh filename=meshes/bent_sealed_tapered_needle2_vhacd.obj scale=0.01 0.01 0.01; visual mesh filename=meshes/bent_sealed_tapered_needle2.obj scale=0.01 0.01 0.01
